File: IMU-pcb/IMU-pcb.kicad_pcb (KiCad board)
At the start: 2 copper layers, 76.8 x 41 mm, 13 parts, among them J1 Status Rails, J2 Battery, J3 AUX Sensor, U1 4056Board, U2 WeMos_D1_mini, U3 IMU Sensor

Commit message: new version of PCB
Connections:
- net D6 renamed RED
- D3 pad 2: D7 -> GND
- D3 pad 3: D8 -> GRN
- D3 pad 4: GND -> BLU
- U2 pad 6: D7 -> GRN
- U2 pad 7: D8 -> BLU
Routing:
- net GRN: track 0.00 -> 61.9 mm
- net D8: track 61.0 -> 0.00 mm
- net BLU: track 0.00 -> 60.9 mm
- net D7: track 58.7 -> 0.00 mm
- net +5V: track 120.2 -> 120.8 mm
Other:
- board text added: "PLANET v1.1.1"
- board text removed: "PLANET v1.1"
Changed lines of the file:
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@@
       (drillshape 0)
       (scaleselection 1)
-      (outputdirectory "C:/Users/angel/Desktop/IMU-pcb/gerbers_v1.1/")
+      (outputdirectory "../gerbers_v1.1.1/")
     )
   )
@@
   (net 9 "SDA")
   (net 10 "INT_PIN2")
-  (net 11 "D7")
-  (net 12 "D8")
+  (net 11 "GRN")
+  (net 12 "BLU")
   (net 13 "unconnected-(U1-Pad6)")
   (net 14 "unconnected-(U3-PadJP1_2)")
@@
   (net 27 "unconnected-(U2-Pad16)")
   (net 28 "+3.3V")
-  (net 29 "D6")
+  (net 29 "RED")
   (net 30 "unconnected-(U2-Pad11)")
   (footprint "PLANETS:JST_PH_S2B-PH-K_02x2.00mm_Angled" (layer "F.Cu")
@@
       (net 7 "Net-(D3-Pad1)") (pintype "passive"))
     (pad "2" thru_hole circle (at 0 3.5 270) (size 2 2) (drill 0.762) (layers *.Cu *.Mask)
-      (net 29 "D6") (pintype "passive"))
+      (net 29 "RED") (pintype "passive"))
     (model "C:/Users/angel/Desktop/IMU-pcb/lib/3D models/resistors.3dshapes/100K.STEP"
       (offset (xyz 0 -1.6 1))
@@
       (net 7 "Net-(D3-Pad1)") (pinfunction "RA") (pintype "passive"))
     (pad "2" thru_hole oval (at 1.27 0) (size 1.07 1.8) (drill 0.9) (layers *.Cu *.Mask)
-      (net 11 "D7") (pinfunction "GA") (pintype "passive"))
+      (net 22 "GND") (pinfunction "GA") (pintype "passive"))
     (pad "3" thru_hole oval (at 2.54 0) (size 1.07 1.8) (drill 0.9) (layers *.Cu *.Mask)
-      (net 12 "D8") (pinfunction "BA") (pintype "passive"))
+      (net 11 "GRN") (pinfunction "BA") (pintype "passive"))
     (pad "4" thru_hole oval (at 3.81 0) (size 1.07 1.8) (drill 0.9) (layers *.Cu *.Mask)
-      (net 22 "GND") (pinfunction "K") (pintype "passive"))
+      (net 12 "BLU") (pinfunction "K") (pintype "passive"))
     (model "${KICAD6_3DMODEL_DIR}/LED_THT.3dshapes/LED_D5.0mm-4_RGB.wrl"
       (offset (xyz 0 0 0))
@@
       (net 15 "INT_PIN1") (pinfunction "D5") (pintype "bidirectional"))
     (pad "5" thru_hole circle locked (at -1.27 -11.43 90) (size 1.8 1.8) (drill 1.016) (layers *.Cu *.Mask)
-      (net 29 "D6") (pinfunction "D6") (pintype "bidirectional"))
+      (net 29 "RED") (pinfunction "D6") (pintype "bidirectional"))
     (pad "6" thru_hole circle locked (at -3.81 -11.43 180) (size 1.8 1.8) (drill 1.016) (layers *.Cu *.Mask)
-      (net 11 "D7") (pinfunction "D7") (pintype "bidirectional"))
+      (net 11 "GRN") (pinfunction "D7") (pintype "bidirectional"))
     (pad "7" thru_hole circle locked (at -6.35 -11.43 90) (size 1.8 1.8) (drill 1.016) (layers *.Cu *.Mask)
-      (net 12 "D8") (pinfunction "D8") (pintype "bidirectional"))
+      (net 12 "BLU") (pinfunction "D8") (pintype "bidirectional"))
     (pad "8" thru_hole circle locked (at -8.89 -11.43 90) (size 1.8 1.8) (drill 1.016) (layers *.Cu *.Mask)
       (net 28 "+3.3V") (pinfunction "3.3V") (pintype "power_out"))
@@
     (effects (font (size 1 1) (thickness 0.15)) (justify mirror))
   )
-  (gr_text "PLANET v1.1" (at 123.5 107.8) (layer "B.SilkS")
+  (gr_text "PLANET v1.1.1\n" (at 123.5 107.8) (layer "B.SilkS")
     (effects (font (size 2.5 2.5) (thickness 0.15)) (justify mirror))
   )
@@
   (segment (start 180.7 78) (end 176.1 73.4) (width 0.25) (layer "B.Cu") (net 10))
   (segment (start 183.8 84.5) (end 180.7 81.4) (width 0.25) (layer "B.Cu") (net 10))
-  (segment (start 162.37 77.185) (end 161.696012 76.511012) (width 0.25) (layer "B.Cu") (net 11))
+  (segment (start 162.8 79.6) (end 163.5 78.9) (width 0.25) (layer "B.Cu") (net 11))
+  (segment (start 158.788988 76.511012) (end 131.011012 76.511012) (width 0.25) (layer "B.Cu") (net 11))
+  (segment (start 158.788988 76.511012) (end 158.811012 76.511012) (width 0.25) (layer "B.Cu") (net 11))
   (segment (start 131.011012 76.511012) (end 112.471012 95.051012) (width 0.25) (layer "B.Cu") (net 11))
-  (segment (start 161.696012 76.511012) (end 131.011012 76.511012) (width 0.25) (layer "B.Cu") (net 11))
-  (segment (start 162.37 78) (end 162.37 77.185) (width 0.25) (layer "B.Cu") (net 11))
-  (segment (start 145.75 80.25) (end 162.75 80.25) (width 0.25) (layer "B.Cu") (net 12))
-  (segment (start 162.75 80.25) (end 163.64 79.36) (width 0.25) (layer "B.Cu") (net 12))
+  (segment (start 158.811012 76.511012) (end 159.8 77.5) (width 0.25) (layer "B.Cu") (net 11))
+  (segment (start 160.4 79.6) (end 162.8 79.6) (width 0.25) (layer "B.Cu") (net 11))
+  (segment (start 159.8 79) (end 160.4 79.6) (width 0.25) (layer "B.Cu") (net 11))
+  (segment (start 159.8 77.5) (end 159.8 79) (width 0.25) (layer "B.Cu") (net 11))
+  (segment (start 163.64 78.76) (end 163.64 78) (width 0.25) (layer "B.Cu") (net 11))
+  (segment (start 161.95 80.25) (end 162.95 80.25) (width 0.25) (layer "B.Cu") (net 12))
   (segment (start 144.7 79.2) (end 145.75 80.25) (width 0.25) (layer "B.Cu") (net 12))
   (segment (start 112.471012 97.591012) (end 130.862024 79.2) (width 0.25) (layer "B.Cu") (net 12))
+  (segment (start 163.45 80.25) (end 164.8 78.9) (width 0.25) (layer "B.Cu") (net 12))
+  (segment (start 145.75 80.25) (end 161.95 80.25) (width 0.25) (layer "B.Cu") (net 12))
   (segment (start 130.862024 79.2) (end 144.7 79.2) (width 0.25) (layer "B.Cu") (net 12))
-  (segment (start 163.64 79.36) (end 163.64 78) (width 0.25) (layer "B.Cu") (net 12))
+  (segment (start 162.95 80.25) (end 163.45 80.25) (width 0.25) (layer "B.Cu") (net 12))
   (segment (start 110.5 101) (end 110.5 93) (width 0.25) (layer "B.Cu") (net 15))
   (segment (start 110.5 91.942024) (end 112.471012 89.971012) (width 0.25) (layer "B.Cu") (net 15))
@@
   (via (at 125.6 87.9) (size 0.8) (drill 0.4) (layers "F.Cu" "B.Cu") (free) (net 22))
   (via (at 118 75.9) (size 0.8) (drill 0.4) (layers "F.Cu" "B.Cu") (free) (net 22))
-  (segment (start 159.75 104.75) (end 139.95 104.75) (width 0.25) (layer "F.Cu") (net 24))
-  (segment (start 112.25 102) (end 111 100.75) (width 0.25) (layer "F.Cu") (net 24))
   (segment (start 163.75 108.75) (end 159.75 104.75) (width 0.25) (layer "F.Cu") (net 24))
-  (segment (start 168.95 79.5) (end 168.95 105.8) (width 0.25) (layer "F.Cu") (net 24))
-  (segment (start 168.95 105.8) (end 166 108.75) (width 0.25) (layer "F.Cu") (net 24))
+  (segment (start 112.25 102) (end 111 100.75) (width 0.25) (layer "F.Cu") (net 24))
+  (segment (start 168.95 79.5) (end 168.95 82.85) (width 0.25) (layer "F.Cu") (net 24))
+  (segment (start 159.75 104.75) (end 139.95 104.75) (width 0.25) (layer "F.Cu") (net 24))
   (segment (start 133.462024 102) (end 112.25 102) (width 0.25) (layer "F.Cu") (net 24))
+  (segment (start 168.95 105.8) (end 166 108.75) (width 0.25) (layer "F.Cu") (net 24))
   (segment (start 111 100.75) (end 111 81.75) (width 0.25) (layer "F.Cu") (net 24))
+  (segment (start 166 108.75) (end 163.75 108.75) (width 0.25) (layer "F.Cu") (net 24))
   (segment (start 139.95 104.75) (end 135.331012 100.131012) (width 0.25) (layer "F.Cu") (net 24))
+  (segment (start 169.7 83.6) (end 169.7 86.1) (width 0.25) (layer "F.Cu") (net 24))
   (segment (start 111 81.75) (end 112.88 79.87) (width 0.25) (layer "F.Cu") (net 24))
+  (segment (start 169.7 86.1) (end 168.95 86.85) (width 0.25) (layer "F.Cu") (net 24))
+  (segment (start 168.95 82.85) (end 169.7 83.6) (width 0.25) (layer "F.Cu") (net 24))
   (segment (start 112.88 79.87) (end 112.88 71.7) (width 0.25) (layer "F.Cu") (net 24))
-  (segment (start 166 108.75) (end 163.75 108.75) (width 0.25) (layer "F.Cu") (net 24))
   (segment (start 135.331012 100.131012) (end 133.462024 102) (width 0.25) (layer "F.Cu") (net 24))
+  (segment (start 168.95 86.85) (end 168.95 105.8) (width 0.25) (layer "F.Cu") (net 24))
   (segment (start 130.082024 74.9) (end 112.471012 92.511012) (width 0.25) (layer "B.Cu") (net 29))
   (segment (start 147.6 74.9) (end 130.082024 74.9) (width 0.25) (layer "B.Cu") (net 29))
