File: IMU-pcb/IMU-pcb.kicad_sch (KiCad schematic)
At the start: 12 parts, among them J1 Conn_01x05_Female, U1 4056Board, U2 WeMos_D1_mini, U3 4754

Commit message: formalized schematic, symbols, and footprints
Parts:
- added J1: Status Rails, bryx-comp-lib:fivePinConn, symbol Connector:Conn_01x05_Female
- J2: renamed from Battery1; value Conn_01x02_Female -> Battery
- J3: renamed from J1; value Conn_01x05_Female -> AUX Sensor
- U3: value 4754 -> IMU Sensor
Connections:
- net 3V3: now also J1.2 (Pin_2)
- net 5V: now also J1.1 (Pin_1)
- net B+: now also J1.4 (Pin_4)
- net B-: now also J1.5 (Pin_5)
- net Switch_GND: now also J1.3 (Pin_3)
Other:
- note added: "AUX Sensor"
- note added: "Battery Connector"
- note added: "D1 Mini"
- note added: "IMU Sensor"
- note added: "Power Protection"
- note added: "Status Rails"
- moved on the sheet: D1, D2, D3, J2, J3, R1, R2, R3, S1, U1, U2, U3

Commit message: working on desktop
Parts:
- D1: footprint LED_THT:LED_D5.0mm -> PLANETS:LED_D5.0mm
- J1: footprint bryx-comp-lib:fivePinConn -> PLANETS:fivePinConn
- J2: footprint Connectors_JST:JST_PH_S2B-PH-K_02x2.00mm_Angled -> PLANETS:JST_PH_S2B-PH-K_02x2.00mm_Angled
- J3: footprint Connectors_JST:JST_XH_S05B-XH-A_05x2.50mm_Angled -> PLANETS:JST_XH_S05B-XH-A_05x2.50mm_Angled
- R1: footprint SlimeVRMotherBoard:18Ω -> PLANETS:18Ω
- R2: footprint SlimeVRMotherBoard:180KΩ -> PLANETS:180KΩ
- R3: footprint SlimeVRMotherBoard:10Ω -> PLANETS:10Ω
- S1: footprint SlimeVRMotherBoard:Wowoone_Slide_Switch_5mm -> PLANETS:Wowoone_Slide_Switch_5mm
- U1: footprint SlimeVRMotherBoard:4056Board -> PLANETS:4056Board
- U2: footprint wemos-d1-mini:wemos-d1-mini-with-pin-header-and-connector -> PLANETS:wemos-d1-mini-with-pin-header-and-connector
- U3: footprint BNO085:BNO085 -> PLANETS:BNO085
Connections:
- net Switch_GND: now also S1.1 (T1); no longer S1.2 (T2)
- net at U1.4 (Out-): now also S1.2 (T2); no longer S1.1 (T1)
Other:
- moved on the sheet: S1
Changed lines of the file:
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@@
       (effects (font (size 1.27 1.27)) (justify left))
     )
-    (property "Footprint" "bryx-comp-lib:fivePinConn" (id 2) (at 139.7 53.086 0)
+    (property "Footprint" "PLANETS:fivePinConn" (id 2) (at 139.7 53.086 0)
       (effects (font (size 1.27 1.27)) hide)
     )
@@
       (effects (font (size 1.27 1.27)) (justify left))
     )
-    (property "Footprint" "Connectors_JST:JST_PH_S2B-PH-K_02x2.00mm_Angled" (id 2) (at 141.224 24.384 0)
+    (property "Footprint" "PLANETS:JST_PH_S2B-PH-K_02x2.00mm_Angled" (id 2) (at 141.224 24.384 0)
       (effects (font (size 1.27 1.27)) hide)
     )
@@
     (property "Reference" "U1" (id 0) (at 43.053 108.7104 0))
     (property "Value" "4056Board" (id 1) (at 43.053 111.2473 0))
-    (property "Footprint" "SlimeVRMotherBoard:4056Board" (id 2) (at 43.053 101.727 0)
+    (property "Footprint" "PLANETS:4056Board" (id 2) (at 43.053 101.727 0)
       (effects (font (size 1.27 1.27)) hide)
     )
@@
       (effects (font (size 1.524 1.524)))
     )
-    (property "Footprint" "wemos-d1-mini:wemos-d1-mini-with-pin-header-and-connector" (id 2) (at 76.327 62.23 0)
+    (property "Footprint" "PLANETS:wemos-d1-mini-with-pin-header-and-connector" (id 2) (at 76.327 62.23 0)
       (effects (font (size 1.524 1.524)))
     )
@@
     (property "Reference" "R1" (id 0) (at 36.957 53.34 90))
     (property "Value" "18" (id 1) (at 36.957 51.1611 90))
-    (property "Footprint" "SlimeVRMotherBoard:18Ω" (id 2) (at 36.957 55.118 90)
+    (property "Footprint" "PLANETS:18Ω" (id 2) (at 36.957 55.118 90)
       (effects (font (size 1.27 1.27)) hide)
     )
@@
       (effects (font (size 1.27 1.27)) (justify left))
     )
-    (property "Footprint" "Connectors_JST:JST_XH_S05B-XH-A_05x2.50mm_Angled" (id 2) (at 175.895 24.511 0)
+    (property "Footprint" "PLANETS:JST_XH_S05B-XH-A_05x2.50mm_Angled" (id 2) (at 175.895 24.511 0)
       (effects (font (size 1.27 1.27)) hide)
     )
@@
     (pin "2")
   )
-  (symbol (lib_id "SlimeVRLibrary:SlideSwitch") (at 63.373 100.457 180) (unit 1)
-    (in_bom yes) (on_board yes)
-    (property "Reference" "S1" (id 0) (at 63.246 101.981 0))
-    (property "Value" "SlideSwitch" (id 1) (at 63.373 104.0329 0))
-    (property "Footprint" "SlimeVRMotherBoard:Wowoone_Slide_Switch_5mm" (id 2) (at 63.373 100.457 0)
+  (symbol (lib_id "SlimeVRLibrary:SlideSwitch") (at 63.373 100.457 0) (unit 1)
+    (in_bom yes) (on_board yes)
+    (property "Reference" "S1" (id 0) (at 63.5 98.933 0))
+    (property "Value" "SlideSwitch" (id 1) (at 63.373 96.8811 0))
+    (property "Footprint" "PLANETS:Wowoone_Slide_Switch_5mm" (id 2) (at 63.373 100.457 0)
       (effects (font (size 1.27 1.27)) hide)
     )
@@
     (property "Reference" "D1" (id 0) (at 45.5295 48.3702 0))
     (property "Value" "LED" (id 1) (at 45.5295 50.9071 0))
-    (property "Footprint" "LED_THT:LED_D5.0mm" (id 2) (at 47.117 53.34 0)
+    (property "Footprint" "PLANETS:LED_D5.0mm" (id 2) (at 47.117 53.34 0)
       (effects (font (size 1.27 1.27)) hide)
     )
@@
     (property "Reference" "R2" (id 0) (at 57.277 40.64 90))
     (property "Value" "180k" (id 1) (at 57.277 38.4611 90))
-    (property "Footprint" "SlimeVRMotherBoard:180KΩ" (id 2) (at 57.277 42.418 90)
+    (property "Footprint" "PLANETS:180KΩ" (id 2) (at 57.277 42.418 90)
       (effects (font (size 1.27 1.27)) hide)
     )
@@
     (property "Reference" "R3" (id 0) (at 57.15 53.34 90))
     (property "Value" "10" (id 1) (at 57.277 51.1611 90))
-    (property "Footprint" "SlimeVRMotherBoard:10Ω" (id 2) (at 57.277 55.118 90)
+    (property "Footprint" "PLANETS:10Ω" (id 2) (at 57.277 55.118 90)
       (effects (font (size 1.27 1.27)) hide)
     )
@@
     (property "Reference" "U3" (id 0) (at 122.047 78.2152 0))
     (property "Value" "IMU Sensor" (id 1) (at 122.047 80.7521 0))
-    (property "Footprint" "BNO085:BNO085" (id 2) (at 122.047 97.155 0)
+    (property "Footprint" "PLANETS:BNO085" (id 2) (at 122.047 97.155 0)
       (effects (font (size 1.27 1.27)) (justify bottom) hide)
     )
@@
   (symbol_instances
     (path "/96d45ffe-e1bf-4f2d-b0c1-7d3af05cd2fd"
-      (reference "D1") (unit 1) (value "LED") (footprint "LED_THT:LED_D5.0mm")
+      (reference "D1") (unit 1) (value "LED") (footprint "PLANETS:LED_D5.0mm")
     )
     (path "/e35e1e49-7866-4359-beb1-015e80952e45"
@@
     )
     (path "/08a5be96-4863-4e23-8756-92b561e669b1"
-      (reference "J1") (unit 1) (value "Status Rails") (footprint "bryx-comp-lib:fivePinConn")
+      (reference "J1") (unit 1) (value "Status Rails") (footprint "PLANETS:fivePinConn")
     )
     (path "/177edf2a-128d-42b9-96c0-90ff94f480d7"
-      (reference "J2") (unit 1) (value "Battery") (footprint "Connectors_JST:JST_PH_S2B-PH-K_02x2.00mm_Angled")
+      (reference "J2") (unit 1) (value "Battery") (footprint "PLANETS:JST_PH_S2B-PH-K_02x2.00mm_Angled")
     )
     (path "/5379bcf9-ffec-4d5e-81b6-c6fbcba09713"
-      (reference "J3") (unit 1) (value "AUX Sensor") (footprint "Connectors_JST:JST_XH_S05B-XH-A_05x2.50mm_Angled")
+      (reference "J3") (unit 1) (value "AUX Sensor") (footprint "PLANETS:JST_XH_S05B-XH-A_05x2.50mm_Angled")
     )
     (path "/42d4a0ee-c15c-46bd-b5d4-70e9c7465a4c"
-      (reference "R1") (unit 1) (value "18") (footprint "SlimeVRMotherBoard:18Ω")
+      (reference "R1") (unit 1) (value "18") (footprint "PLANETS:18Ω")
     )
     (path "/ad24cb45-f6bb-42de-a0e5-d559433b1b4f"
-      (reference "R2") (unit 1) (value "180k") (footprint "SlimeVRMotherBoard:180KΩ")
+      (reference "R2") (unit 1) (value "180k") (footprint "PLANETS:180KΩ")
     )
     (path "/c08e599e-c337-4bf8-b61d-04238fec98d3"
-      (reference "R3") (unit 1) (value "10") (footprint "SlimeVRMotherBoard:10Ω")
+      (reference "R3") (unit 1) (value "10") (footprint "PLANETS:10Ω")
     )
     (path "/8bc4c9ea-311b-44b8-97ff-03520d1dcd65"
-      (reference "S1") (unit 1) (value "SlideSwitch") (footprint "SlimeVRMotherBoard:Wowoone_Slide_Switch_5mm")
+      (reference "S1") (unit 1) (value "SlideSwitch") (footprint "PLANETS:Wowoone_Slide_Switch_5mm")
     )
     (path "/22ee0647-68d7-4c07-ad73-6d28cf15eb9d"
-      (reference "U1") (unit 1) (value "4056Board") (footprint "SlimeVRMotherBoard:4056Board")
+      (reference "U1") (unit 1) (value "4056Board") (footprint "PLANETS:4056Board")
     )
     (path "/3a5913aa-9933-403e-ac9e-6496251c88c9"
-      (reference "U2") (unit 1) (value "WeMos_D1_mini") (footprint "wemos-d1-mini:wemos-d1-mini-with-pin-header-and-connector")
+      (reference "U2") (unit 1) (value "WeMos_D1_mini") (footprint "PLANETS:wemos-d1-mini-with-pin-header-and-connector")
     )
     (path "/e375db96-9775-488a-b860-a5964ea556b5"
-      (reference "U3") (unit 1) (value "IMU Sensor") (footprint "BNO085:BNO085")
-    )
-  )
+      (reference "U3") (unit 1) (value "IMU Sensor") (footprint "PLANETS:BNO085")
+    )
+  )

Commit message: Finished v1.1 layout
Parts:
- removed D1: LED, PLANETS:LED_D5.0mm, symbol Device:LED
- removed R1: 18, PLANETS:18Ω, symbol Device:R
- removed R3: 10, PLANETS:10Ω, symbol Device:R
- added D3: LED_RGBK, LED_THT:LED_D5.0mm-4_RGB, symbol Device:LED_RGBK
- added R2: 150, PLANETS:150Ω, symbol Device:R
- renumbered D2 to D1, D3 to D2, R2 to R1
Connections:
- net INT_PIN2: now also U2.3 (D0); no longer U2.5 (D6)
- net SCL: now also J3.4 (Pin_4); no longer J3.3 (Pin_3)
- net SDA: now also J3.3 (Pin_3); no longer J3.4 (Pin_4)
- net at S1.2 (T2): now also D1.1 (K), D2.1 (K); no longer U1.4 (Out-)
- net D7: now reaches U2.6 (D7)
- net D7: now also D3.2 (GA)
- net D8: now reaches U2.7 (D8)
- net D8: now also D3.3 (BA)
- net 3V3 renamed +3.3V
- net 5V renamed +5V
- net +5V: now also S1.1 (T1); no longer D1.1 (K), D2.1 (K)
- net Switch_GND renamed GND
- net GND: now also U1.4 (Out-), D3.4 (K); no longer S1.1 (T1)
- new net: D3.1 (RA), R2.1
- new net D6: R2.2, U2.5 (D6)
- no-connect marks 14 -> 12
Other:
- note added: "RBG LED"
- title: IMU-pcb -> PLANET
- moved on the sheet: D1, D2, J1, J2, R1, S1, U1, U2

Commit message: Adjusted pcb layout to be better
Parts:
- R1: footprint PLANETS:180KΩ -> PLANETS:180KOhm
- R2: footprint PLANETS:150Ω -> PLANETS:150Ohm
Changed lines of the file:
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@@
     (property "Reference" "R2" (id 0) (at 177.8 43.5442 90))
     (property "Value" "150" (id 1) (at 177.8 46.0811 90))
-    (property "Footprint" "PLANETS:150Ω" (id 2) (at 177.8 50.038 90)
+    (property "Footprint" "PLANETS:150Ohm" (id 2) (at 177.8 50.038 90)
       (effects (font (size 1.27 1.27)) hide)
     )
@@
     (property "Reference" "R1" (id 0) (at 44.577 34.29 90))
     (property "Value" "180k" (id 1) (at 44.577 32.1111 90))
-    (property "Footprint" "PLANETS:180KΩ" (id 2) (at 44.577 36.068 90)
+    (property "Footprint" "PLANETS:180KOhm" (id 2) (at 44.577 36.068 90)
       (effects (font (size 1.27 1.27)) hide)
     )
@@
     )
     (path "/ad24cb45-f6bb-42de-a0e5-d559433b1b4f"
-      (reference "R1") (unit 1) (value "180k") (footprint "PLANETS:180KΩ")
+      (reference "R1") (unit 1) (value "180k") (footprint "PLANETS:180KOhm")
     )
     (path "/2536c513-bcfb-4e03-8ff8-03250600c11f"
-      (reference "R2") (unit 1) (value "150") (footprint "PLANETS:150Ω")
+      (reference "R2") (unit 1) (value "150") (footprint "PLANETS:150Ohm")
     )
     (path "/8bc4c9ea-311b-44b8-97ff-03520d1dcd65"

Commit message: new version of PCB
Connections:
- net GND: now also D3.2 (GA); no longer D3.4 (K)
- net D6 renamed RED
- net D7 renamed GRN
- net GRN: now also D3.3 (BA); no longer D3.2 (GA)
- net D8 renamed BLU
- net BLU: now also D3.4 (K); no longer D3.3 (BA)
Changed lines of the file:
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@@
     (stroke (width 0) (type default) (color 0 0 0 0))
   )
-  (polyline (pts (xy 190.5 69.469) (xy 190.5 33.02))
-    (stroke (width 0) (type default) (color 0 0 0 0))
-  )
-  (polyline (pts (xy 190.5 12.065) (xy 190.5 32.893))
+  (polyline (pts (xy 191.77 69.469) (xy 191.77 32.893))
+    (stroke (width 0) (type default) (color 0 0 0 0))
+  )
+  (polyline (pts (xy 191.77 12.065) (xy 191.77 32.893))
     (stroke (width 0) (type default) (color 0 0 0 0))
   )
@@
     (stroke (width 0) (type default) (color 0 0 0 0))
   )
-  (polyline (pts (xy 152.4 69.469) (xy 190.5 69.469))
+  (polyline (pts (xy 152.4 69.469) (xy 191.77 69.469))
     (stroke (width 0) (type default) (color 0 0 0 0))
   )
@@
     (stroke (width 0) (type default) (color 0 0 0 0))
   )
-  (polyline (pts (xy 152.4 32.893) (xy 190.5 32.893))
+  (polyline (pts (xy 152.4 32.893) (xy 191.77 32.893))
     (stroke (width 0) (type default) (color 0 0 0 0))
   )
@@
     )
   )
-  (global_label "D6" (shape input) (at 50.8 41.91 180) (fields_autoplaced)
-    (effects (font (size 1.27 1.27)) (justify right))
-    (property "Intersheet References" "${INTERSHEET_REFS}" (id 0) (at 45.9074 41.8306 0)
+  (global_label "RED" (shape input) (at 50.8 41.91 180) (fields_autoplaced)
+    (effects (font (size 1.27 1.27)) (justify right))
+    (property "Intersheet References" "${INTERSHEET_REFS}" (id 0) (at 44.6979 41.8306 0)
       (effects (font (size 1.27 1.27)) (justify right) hide)
     )
@@
     )
   )
-  (global_label "D8" (shape input) (at 50.8 46.99 180) (fields_autoplaced)
-    (effects (font (size 1.27 1.27)) (justify right))
-    (property "Intersheet References" "${INTERSHEET_REFS}" (id 0) (at 45.9074 46.9106 0)
-      (effects (font (size 1.27 1.27)) (justify right) hide)
-    )
-  )
-  (global_label "D6" (shape input) (at 184.15 48.26 0) (fields_autoplaced)
+  (global_label "BLU" (shape input) (at 50.8 46.99 180) (fields_autoplaced)
+    (effects (font (size 1.27 1.27)) (justify right))
+    (property "Intersheet References" "${INTERSHEET_REFS}" (id 0) (at 44.7583 46.9106 0)
+      (effects (font (size 1.27 1.27)) (justify right) hide)
+    )
+  )
+  (global_label "RED" (shape input) (at 184.15 48.26 0) (fields_autoplaced)
     (effects (font (size 1.27 1.27)) (justify left))
-    (property "Intersheet References" "${INTERSHEET_REFS}" (id 0) (at 189.0426 48.1806 0)
+    (property "Intersheet References" "${INTERSHEET_REFS}" (id 0) (at 190.2521 48.1806 0)
       (effects (font (size 1.27 1.27)) (justify left) hide)
     )
   )
-  (global_label "D7" (shape input) (at 50.8 44.45 180) (fields_autoplaced)
-    (effects (font (size 1.27 1.27)) (justify right))
-    (property "Intersheet References" "${INTERSHEET_REFS}" (id 0) (at 45.9074 44.3706 0)
+  (global_label "GRN" (shape input) (at 50.8 44.45 180) (fields_autoplaced)
+    (effects (font (size 1.27 1.27)) (justify right))
+    (property "Intersheet References" "${INTERSHEET_REFS}" (id 0) (at 44.5164 44.3706 0)
       (effects (font (size 1.27 1.27)) (justify right) hide)
     )
@@
     )
   )
-  (global_label "D7" (shape input) (at 171.45 53.34 0) (fields_autoplaced)
+  (global_label "GRN" (shape input) (at 171.45 58.42 0) (fields_autoplaced)
     (effects (font (size 1.27 1.27)) (justify left))
-    (property "Intersheet References" "${INTERSHEET_REFS}" (id 0) (at 176.3426 53.2606 0)
+    (property "Intersheet References" "${INTERSHEET_REFS}" (id 0) (at 177.7336 58.3406 0)
       (effects (font (size 1.27 1.27)) (justify left) hide)
     )
@@
     )
   )
-  (global_label "D8" (shape input) (at 171.45 58.42 0) (fields_autoplaced)
-    (effects (font (size 1.27 1.27)) (justify left))
-    (property "Intersheet References" "${INTERSHEET_REFS}" (id 0) (at 176.3426 58.3406 0)
-      (effects (font (size 1.27 1.27)) (justify left) hide)
+  (global_label "BLU" (shape input) (at 161.29 53.34 180) (fields_autoplaced)
+    (effects (font (size 1.27 1.27)) (justify right))
+    (property "Intersheet References" "${INTERSHEET_REFS}" (id 0) (at 155.2483 53.2606 0)
+      (effects (font (size 1.27 1.27)) (justify right) hide)
     )
   )
@@
     (pin "4")
   )
-  (symbol (lib_id "power:GND") (at 161.29 53.34 270) (unit 1)
-    (in_bom yes) (on_board yes) (fields_autoplaced)
-    (property "Reference" "#PWR011" (id 0) (at 154.94 53.34 0)
-      (effects (font (size 1.27 1.27)) hide)
-    )
-    (property "Value" "GND" (id 1) (at 158.1151 53.7738 90)
+  (symbol (lib_id "power:GND") (at 171.45 53.34 90) (unit 1)
+    (in_bom yes) (on_board yes) (fields_autoplaced)
+    (property "Reference" "#PWR011" (id 0) (at 177.8 53.34 0)
+      (effects (font (size 1.27 1.27)) hide)
+    )
+    (property "Value" "GND" (id 1) (at 174.625 53.7738 90)
       (effects (font (size 1.27 1.27)) (justify right))
     )
-    (property "Footprint" "" (id 2) (at 161.29 53.34 0)
-      (effects (font (size 1.27 1.27)) hide)
-    )
-    (property "Datasheet" "" (id 3) (at 161.29 53.34 0)
-      (effects (font (size 1.27 1.27)) hide)
-    )
+    (property "Footprint" "" (id 2) (at 171.45 53.34 0)
+      (effects (font (size 1.27 1.27)) hide)
+    )
+    (property "Datasheet" "" (id 3) (at 171.45 53.34 0)
+      (effects (font (size 1.27 1.27)) hide)
+    )
